File: _autosave-interface_panel.kicad_sch (KiCad schematic)
At the start: 8 parts, among them J1 Conn_02x04_Odd_Even

Commit message: display and overall layout changed
Parts:
- oled1: footprint oled0.9in:SSD1306-0.91-OLED-4pin-128x32 -> oled0.9in:MODULE_DM-OLED096-636
Changed lines of the file:
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@@
 			)
 		)
-		(property "Footprint" "oled0.9in:SSD1306-0.91-OLED-4pin-128x32"
+		(property "Footprint" "oled0.9in:MODULE_DM-OLED096-636"
 			(at 72.136 107.696 0)
 			(effects

Commit message: changed layout with 12mm push_but
Parts:
- 0/1, H-1, H-2: footprint Button_Switch_THT:SW_PUSH_6mm -> pushbutt_12x12x7.3:SW_TS14-1212-140-BK-160-SCR-D
Changed lines of the file:
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@@
 			)
 		)
-		(property "Footprint" "Button_Switch_THT:SW_PUSH_6mm"
+		(property "Footprint" "pushbutt_12x12x7.3:SW_TS14-1212-140-BK-160-SCR-D"
 			(at 135.89 48.26 0)
 			(effects
@@
 			)
 		)
-		(property "Footprint" "Button_Switch_THT:SW_PUSH_6mm"
+		(property "Footprint" "pushbutt_12x12x7.3:SW_TS14-1212-140-BK-160-SCR-D"
 			(at 166.37 49.53 0)
 			(effects
@@
 			)
 		)
-		(property "Footprint" "Button_Switch_THT:SW_PUSH_6mm"
+		(property "Footprint" "pushbutt_12x12x7.3:SW_TS14-1212-140-BK-160-SCR-D"
 			(at 152.4 49.53 0)
 			(effects
