File: _autosave-interface_panel.kicad_sch (KiCad schematic)
At the start: 20 parts, among them J1 Conn_02x04_Odd_Even, J2 but1, J3 but2, J4 but3, J5 Led, U2 ATmega328P-P, Y1 Crystal

Commit message: production change-2
Parts:
- H1, H2, H3, H4: footprint (none) -> MountingHole:MountingHole_2.2mm_M2
Changed lines of the file:
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@@
 			)
 		)
-		(property "Footprint" ""
+		(property "Footprint" "MountingHole:MountingHole_2.2mm_M2"
 			(at 137.16 149.86 0)
 			(effects
@@
 			)
 		)
-		(property "Footprint" ""
+		(property "Footprint" "MountingHole:MountingHole_2.2mm_M2"
 			(at 137.16 134.62 0)
 			(effects
@@
 			)
 		)
-		(property "Footprint" ""
+		(property "Footprint" "MountingHole:MountingHole_2.2mm_M2"
 			(at 137.16 157.48 0)
 			(effects
@@
 			)
 		)
-		(property "Footprint" ""
+		(property "Footprint" "MountingHole:MountingHole_2.2mm_M2"
 			(at 137.16 142.24 0)
 			(effects
