File: interface_panel.kicad_sch (KiCad schematic)
At the start: 48 parts, among them J1 Conn_01x04_Pin, J7 Conn_02x05_Odd_Even, J8 `, Q1 BC547, Q2 BC547, U1 SM420561N, U3 ATmega328P-A, U4 SM420561N, U7 TTP223-BA6, U8 TTP223-BA6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

Commit message: fully routed with TH-atmega
Parts:
- removed U3: ATmega328P-A, Package_QFP:TQFP-32_7x7mm_P0.8mm, symbol MCU_Microchip_ATmega:ATmega328P-A
- added U2: ATmega328P-P, Package_DIP:DIP-28_W7.62mm, symbol MCU_Microchip_ATmega:ATmega328P-P
- C1, C2: footprint Capacitor_SMD:C_1206_3216Metric_Pad1.33x1.80mm_HandSolder -> Capacitor_THT:C_Disc_D3.0mm_W2.0mm_P2.50mm
- Y1: footprint Crystal:Crystal_SMD_HC49-SD -> Crystal:Crystal_HC49-U_Vertical
Connections:
- net 5V: now also U2.20 (AVCC), U2.7 (VCC)
- net A4: now also U2.27 (PC4)
- net A5: now also U2.28 (PC5)
- net D13: now also U2.19 (PB5)
- net GND: now also U2.22 (GND), U2.8 (GND)
- net RX: now also U2.2 (PD0)
- net TX: now also U2.3 (PD1)
- net miso: now also U2.18 (PB4)
- net mosi: now also U2.17 (PB3)
- net reset: now also U2.1 (~{RESET}/PC6)
- net at R5.1: now also U2.15 (PB1)
- net at C1.1, Y1.2: now also U2.9 (XTAL1/PB6)
- net at R11.1: now also U2.13 (PD7)
- net at R7.1: now also U2.5 (PD3)
- net at R8.1: now also U2.6 (PD4)
- net at R10.1: now also U2.12 (PD6)
- net at R12.1: now also U2.14 (PB0)
- net at R3.1: now also U2.16 (PB2)
- net at R6.1: now also U2.4 (PD2)
- net at C2.1, Y1.1: now also U2.10 (XTAL2/PB7)
- net at R9.1: now also U2.11 (PD5)
Changed lines of the file:
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@@
 	)
 	(symbol
+		(lib_id "MCU_Microchip_ATmega:ATmega328P-P")
+		(at 213.36 66.04 0)
+		(unit 1)
+		(exclude_from_sim no)
+		(in_bom yes)
+		(on_board yes)
+		(dnp no)
+		(fields_autoplaced yes)
+		(property "Reference" "U2"
+			(at 191.77 29.1398 0)
+			(effects
+				(font
+					(size 1.27 1.27)
+				)
+			)
+		)
+		(property "Value" "ATmega328P-P"
+			(at 191.77 31.6798 0)
+			(effects
+				(font
+					(size 1.27 1.27)
+				)
+			)
+		)
+		(property "Footprint" "Package_DIP:DIP-28_W7.62mm"
+			(at 213.36 66.04 0)
+			(effects
+				(font
+					(size 1.27 1.27)
+					(italic yes)
+				)
+				(hide yes)
+			)
+		)
+		(property "Datasheet" "http://ww1.microchip.com/downloads/en/DeviceDoc/ATmega328_P%20AVR%20MCU%20with%20picoPower%20Technology%20Data%20Sheet%2040001984A.pdf"
+			(at 213.36 66.04 0)
+			(effects
+				(font
+					(size 1.27 1.27)
+				)
+				(hide yes)
+			)
+		)
+		(property "Description" "20MHz, 32kB Flash, 2kB SRAM, 1kB EEPROM, DIP-28"
+			(at 213.36 66.04 0)
+			(effects
+				(font
+					(size 1.27 1.27)
+				)
+				(hide yes)
+			)
+		)
+		(pin "21"
+		)
+		(pin "7"
+		)
+		(pin "6"
+		)
+		(pin "12"
+		)
+		(pin "17"
+		)
+		(pin "28"
+		)
+		(pin "18"
+		)
+		(pin "19"
+		)
+		(pin "20"
+		)
+		(pin "26"
+		)
+		(pin "3"
+		)
+		(pin "13"
+		)
+		(pin "2"
+		)
+		(pin "22"
+		)
+		(pin "9"
+		)
+		(pin "23"
+		)
+		(pin "24"
+		)
+		(pin "1"
+		)
+		(pin "8"
+		)
+		(pin "5"
+		)
+		(pin "15"
+		)
+		(pin "14"
+		)
+		(pin "16"
+		)
+		(pin "10"
+		)
+		(pin "25"
+		)
+		(pin "27"
+		)
+		(pin "4"
+		)
+		(pin "11"
+		)
+		(instances
+			(project ""
+				(path "/9f0ac2f5-026e-46a7-84a3-e69ffa4f4cba"
+					(reference "U2")
+					(unit 1)
+				)
+			)
+		)
+	)
+	(symbol
 		(lib_id "power:GND")
 		(at 213.36 107.95 0)
@@
 			)
 		)
-		(property "Footprint" "Capacitor_SMD:C_1206_3216Metric_Pad1.33x1.80mm_HandSolder"
+		(property "Footprint" "Capacitor_THT:C_Disc_D3.0mm_W2.0mm_P2.50mm"
 			(at 248.92 48.5648 0)
 			(effects
@@
 	)
 	(symbol
-		(lib_id "MCU_Microchip_ATmega:ATmega328P-A")
-		(at 213.36 66.04 0)
-		(unit 1)
-		(exclude_from_sim no)
-		(in_bom yes)
-		(on_board yes)
-		(dnp no)
-		(fields_autoplaced yes)
-		(property "Reference" "U3"
-			(at 215.5033 104.14 0)
-			(effects
-				(font
-					(size 1.27 1.27)
-				)
-				(justify left)
-			)
-		)
-		(property "Value" "ATmega328P-A"
-			(at 215.5033 106.68 0)
-			(effects
-				(font
-					(size 1.27 1.27)
-				)
-				(justify left)
-			)
-		)
-		(property "Footprint" "Package_QFP:TQFP-32_7x7mm_P0.8mm"
-			(at 213.36 66.04 0)
-			(effects
-				(font
-					(size 1.27 1.27)
-					(italic yes)
-				)
-				(hide yes)
-			)
-		)
-		(property "Datasheet" "http://ww1.microchip.com/downloads/en/DeviceDoc/ATmega328_P%20AVR%20MCU%20with%20picoPower%20Technology%20Data%20Sheet%2040001984A.pdf"
-			(at 213.36 66.04 0)
-			(effects
-				(font
-					(size 1.27 1.27)
-				)
-				(hide yes)
-			)
-		)
-		(property "Description" "20MHz, 32kB Flash, 2kB SRAM, 1kB EEPROM, TQFP-32"
-			(at 213.36 66.04 0)
-			(effects
-				(font
-					(size 1.27 1.27)
-				)
-				(hide yes)
-			)
-		)
-		(pin "26"
-		)
-		(pin "14"
-		)
-		(pin "16"
-		)
-		(pin "31"
-		)
-		(pin "28"
-		)
-		(pin "1"
-		)
-		(pin "21"
-		)
-		(pin "32"
-		)
-		(pin "3"
-		)
-		(pin "18"
-		)
-		(pin "13"
-		)
-		(pin "25"
-		)
-		(pin "20"
-		)
-		(pin "5"
-		)
-		(pin "23"
-		)
-		(pin "15"
-		)
-		(pin "19"
-		)
-		(pin "8"
-		)
-		(pin "4"
-		)
-		(pin "6"
-		)
-		(pin "22"
-		)
-		(pin "12"
-		)
-		(pin "17"
-		)
-		(pin "7"
-		)
-		(pin "24"
-		)
-		(pin "27"
-		)
-		(pin "29"
-		)
-		(pin "30"
-		)
-		(pin "2"
-		)
-		(pin "10"
-		)
-		(pin "11"
-		)
-		(pin "9"
-		)
-		(instances
-			(project ""
-				(path "/9f0ac2f5-026e-46a7-84a3-e69ffa4f4cba"
-					(reference "U3")
-					(unit 1)
-				)
-			)
-		)
-	)
-	(symbol
 		(lib_id "Device:R")
 		(at 234.95 93.98 90)
@@
 			)
 		)
-		(property "Footprint" "Crystal:Crystal_SMD_HC49-SD"
+		(property "Footprint" "Crystal:Crystal_HC49-U_Vertical"
 			(at 237.49 53.34 0)
 			(effects
@@
 			)
 		)
-		(property "Footprint" "Capacitor_SMD:C_1206_3216Metric_Pad1.33x1.80mm_HandSolder"
+		(property "Footprint" "Capacitor_THT:C_Disc_D3.0mm_W2.0mm_P2.50mm"
 			(at 248.92 56.1848 0)
 			(effects
