File: interface_panel.kicad_sch (KiCad schematic)
At the start: 48 parts, among them J1 Conn_01x04_Pin, J7 Conn_02x05_Odd_Even, J8 `, Q1 BC547, Q2 BC547, U1 SM420561N, U3 ATmega328P-A, U4 SM420561N, U7 TTP223-BA6, U8 TTP223-BA6, U9 TTP223-BA6, Y1 Crystal

Commit message: updated as on 03-04-26
Parts:
- removed C6, C7, C8: C, Capacitor_SMD:C_1206_3216Metric_Pad1.33x1.80mm_HandSolder, symbol Device:C
- removed D5, D6, D7: LED, PCM_SparkFun-LED:LED_1206_3216Metric, symbol PCM_SparkFun-LED:LED
- removed J1: Conn_01x04_Pin, Connector_FFC-FPC:Amphenol_F32Q-1A7x1-11004_1x04-1MP_P0.5mm_Horizontal, symbol Connector:Conn_01x04_Pin
- removed Q2: BC547, Package_TO_SOT_THT:TO-92_Inline, symbol Transistor_BJT:BC547
- removed R14, R18, R20, R23: R, Resistor_SMD:R_1206_3216Metric_Pad1.30x1.75mm_HandSolder, symbol Device:R
- removed R19, R21, R22: 10k, Resistor_SMD:R_1206_3216Metric_Pad1.30x1.75mm_HandSolder, symbol Device:R
- removed U4: SM420561N, Display_7Segment:7SegmentLED_LTS6760_LTS6780, symbol Display_Character:SM420561N
- removed U7, U8, U9: TTP223-BA6, TTP223-BA6:SOT23-6, symbol TTP223:TTP223-BA6
- added J1: pot_con, Connector_JST:JST_EH_B3B-EH-A_1x03_P2.50mm_Vertical, symbol Connector:Conn_01x03_Pin
- added LED1: LED_5x5mm, PCM_LED_THT_AKL:LED_Rectangular_W5.0mm_H5.0mm, symbol PCM_LED_AKL:LED_5x5mm
- added RV1: R_Potentiometer, pot:PTV09, symbol Device:R_Potentiometer
- J8: footprint Connector_PinHeader_2.54mm:PinHeader_2x03_P2.54mm_Vertical -> Connector_JST:JST_EH_B6B-EH-A_1x06_P2.50mm_Vertical
Connections:
- net 5V: now also J1.1 (Pin_1), RV1.1
- net GND: now also J8.5 (Pin_5), J1.3 (Pin_3), LED1.1 (K), RV1.3; no longer J8.4 (Pin_4)
- net S. LED: now also R4.1
- net mosi: now also J8.4 (Pin_4); no longer J8.5 (Pin_5), R4.1
- net reset: now also J8.1 (Pin_1); no longer J8.2 (Pin_2)
- net A4: no longer names the net of U3.27 (PC4)
- net A4: no longer J7.10 (Pin_10)
- net A5: no longer names the net of U3.28 (PC5)
- net A5: no longer J7.9 (Pin_9)
- net CC2: no longer names the net of R4.2
- net CC2: now also LED1.2 (A)
- net D13 renamed sck
- net sck: now also J8.2 (Pin_2); no longer J8.1 (Pin_1)
- new net lamp: J1.2 (Pin_2), J7.10 (Pin_10), RV1.2
- no-connect marks 6 -> 8
Other:
- moved on the sheet: B2, D1, PWR1, R1
